File: samd21_breakout.sch (KiCad schematic (older format))
At the start: 36 parts, among them J1 USB_A, J2 SWD, J3 Conn_02x07_Odd_Even, SW1 RESET, SW2 BOOTL, SW3 USR, U1 ATSAMD21G16A, U2 XC6206P332MR, Y1 16MHz

Commit message: Add readme, images, schematic, and update the USB symbol
Parts:
- J1: symbol Connector_Specialized:USB_A -> Connector:USB_A
Changed lines of the file:
@@
 EESchema Schematic File Version 4
 LIBS:samd21_breakout-cache
-EELAYER 26 0
+EELAYER 29 0
 EELAYER END
 $Descr A4 11693 8268
@@
 $EndComp
 $Comp
-L Connector_Specialized:USB_A J1
+L Connector:USB_A J1
 U 1 1 5AA52E87
 P 1200 2300
